File: romeo-pcb.kicad_pcb (KiCad board)
At the start: 2 copper layers, 247.6 x 99.2 mm, 138 parts, among them J1 AVR-ISP-6, SW0 KEYSW, SW1 KEYSW, SW10 KEYSW, SW11 KEYSW, SW12 KEYSW, SW13 KEYSW, SW14 KEYSW, SW15 KEYSW, SW16 KEYSW, SW17 KEYSW, SW18 KEYSW, SW19 KEYSW, SW2 KEYSW, SW20 KEYSW, SW21 KEYSW, SW22 KEYSW, SW23 KEYSW, SW24 KEYSW, SW25 KEYSW, SW26 KEYSW, SW27 KEYSW, SW28 KEYSW, SW29 KEYSW, SW3 KEYSW, SW30 KEYSW, SW31 KEYSW, SW32 KEYSW, SW33 KEYSW, SW34 KEYSW, SW35 KEYSW, SW36 KEYSW, SW37 KEYSW, SW38 KEYSW, SW39 KEYSW, SW4 KEYSW, SW40 KEYSW, SW41 KEYSW, SW42 KEYSW, SW43 KEYSW, SW44 KEYSW, SW45 KEYSW, SW46 KEYSW, SW47 KEYSW, SW5 KEYSW, SW6 KEYSW, SW7 KEYSW, SW8 KEYSW, SW9 KEYSW, U1 ATmega328P-PU, Y1 Crystal

Commit message: update
Parts:
- removed BOOT1: BOOT, cftkb:SW_PUSH_6mm
- removed C1, C2: 22p, cftkb:C_Disc_D3.0mm_W1.6mm_P2.50mm
- removed C3: 4.7u, cftkb:CP_Radial_D4.0mm_P1.50mm
- removed C4, C5: 0.1u, cftkb:C_Disc_D4.3mm_W1.9mm_P5.00mm
- removed D45, D46: 3.6V, cftkb:D_DO-35_SOD27_P5.08mm_Horizontal
- removed F1: 100mA, cftkb:polyfuse_5.1mm
- removed the G*** at (115.0, 136.9) (x2)
- removed the G*** at (176.1, 101.8)
- removed the G*** at (127.3, 131.5) (x2)
- removed the G*** at (161.8, 133.0) (x2)
- removed the G*** at (188.3, 123.5)
- removed the G*** at (176.0, 118.1)
- removed J1: AVR-ISP-6, cftkb:AVR_ICSP_3x2
- removed LED1: POWER, cftkb:LED_D3.0mm
- removed R1, R7: 1.5K, Resistor_THT:R_Axial_DIN0204_L3.6mm_D1.6mm_P5.08mm_Horizontal
- removed R2, R3: 5.1K, Resistor_THT:R_Axial_DIN0204_L3.6mm_D1.6mm_P5.08mm_Horizontal
- removed R4, R5: 75R, Resistor_THT:R_Axial_DIN0204_L3.6mm_D1.6mm_P5.08mm_Horizontal
- removed R6: 10K, Resistor_THT:R_Axial_DIN0204_L3.6mm_D1.6mm_P5.08mm_Horizontal
- removed U1: ATmega328P-PU, Package_DIP:DIP-28_W7.62mm
- removed USB1: USB_C_GCT_USB4085, cftkb:USB_C_GCT_USB4085
- removed Y1: Crystal, cftkb:Crystal_HC49-4H_Vertical
Routing:
- net row1: track 332.3 -> 160.3 mm, vias 3 -> 1
- net row2: track 314.8 -> 144.2 mm, vias 4 -> 1
- net +5V: track 164.7 -> 0.00 mm
- net boot: track 101.2 -> 0.00 mm, vias 2 -> 0
- net reset: track 95.7 -> 0.00 mm, vias 3 -> 0
- net row3: track 228.0 -> 138.1 mm, vias 2 -> 1
- net row0: track 256.9 -> 175.2 mm, vias 2 -> 1
- net sck: track 80.8 -> 0.00 mm, vias 1 -> 0
- net Net-(D45-Pad1): track 47.3 -> 0.00 mm, vias 1 -> 0
- net Net-(D46-Pad1): track 40.5 -> 0.00 mm, vias 1 -> 0
- net GND: track 33.2 -> 0.00 mm, vias 8 -> 2
- net Net-(R3-Pad2): track 31.3 -> 0.00 mm
- net col1: track 203.1 -> 180.4 mm
- net col7: track 94.2 -> 73.1 mm
- net col0: track 236.6 -> 216.6 mm
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- removed copper zone on B.Cu, net GND
- removed copper zone on F.Cu, net GND
Other:
- board text removed: "ATmega328P-PU"
- board text removed: "GND"
- board text removed: "ISP"
- board text removed: "ZENER DIODES"
