File: juliet-pcb.sch (KiCad schematic (older format))
At the start: 114 parts, among them J1 AVR-ISP-6, SW0 KEYSW, SW1 KEYSW, SW10 KEYSW, SW11 KEYSW, SW12 KEYSW, SW13 KEYSW, SW14 KEYSW, SW15 KEYSW, SW16 KEYSW, SW17 KEYSW, SW18 KEYSW, SW19 KEYSW, SW2 KEYSW, SW20 KEYSW, SW21 KEYSW, SW22 KEYSW, SW23 KEYSW, SW24 KEYSW, SW25 KEYSW, SW26 KEYSW, SW27 KEYSW, SW28 KEYSW, SW29 KEYSW, SW3 KEYSW, SW30 KEYSW, SW31 KEYSW, SW32 KEYSW, SW33 KEYSW, SW34 KEYSW, SW35 KEYSW, SW36 KEYSW, SW37 KEYSW, SW38 KEYSW, SW39 KEYSW, SW4 KEYSW, SW40 KEYSW, SW41 KEYSW, SW42 KEYSW, SW43 KEYSW, SW44 KEYSW, SW45 KEYSW, SW46 KEYSW, SW47 KEYSW, SW5 KEYSW, SW6 KEYSW, SW7 KEYSW, SW8 KEYSW, SW9 KEYSW, U1 ATmega328P-PU, Y1 Crystal

Commit message: Updated
Parts:
- removed BOOT1: BOOT, cftkb:SW_PUSH_6mm, symbol romeo-pcb-rescue:SW_PUSH-keyboard_parts
- removed C1, C2: 22p, cftkb:C_Disc_D3.0mm_W1.6mm_P2.50mm, symbol Device:C_Small
- removed C3: 4.7u, cftkb:CP_Radial_D4.0mm_P1.50mm, symbol Device:CP1_Small
- removed C4, C5: 0.1u, cftkb:C_Disc_D4.3mm_W1.9mm_P5.00mm, symbol Device:C_Small
- removed D45, D46: 3.6V, cftkb:D_DO-35_SOD27_P5.08mm_Horizontal, symbol Device:D_Zener_Small
- removed F1: 500mA, cftkb:polyfuse_5.1mm, symbol Device:Polyfuse_Small
- removed J1: AVR-ISP-6, cftkb:AVR_ICSP_3x2, symbol romeo-pcb-rescue:AVR-ISP-6-Connector
- removed LED1: POWER, cftkb:LED_D3.0mm, symbol Device:LED
- removed R1, R7: 1.5K, Resistor_THT:R_Axial_DIN0204_L3.6mm_D1.6mm_P5.08mm_Horizontal, symbol Device:R_Small
- removed R2, R3: 5.1K, Resistor_THT:R_Axial_DIN0204_L3.6mm_D1.6mm_P5.08mm_Horizontal, symbol Device:R_Small
- removed R4, R5: 75R, Resistor_THT:R_Axial_DIN0204_L3.6mm_D1.6mm_P5.08mm_Horizontal, symbol Device:R_Small
- removed R6: 10K, Resistor_THT:R_Axial_DIN0204_L3.6mm_D1.6mm_P5.08mm_Horizontal, symbol Device:R_Small
- removed U1: ATmega328P-PU, Package_DIP:DIP-28_W7.62mm, symbol romeo-pcb-rescue:ATmega328P-PU-MCU_Microchip_ATmega
- removed USB1: USB_C_GCT_USB4085, cftkb:USB_C_GCT_USB4085, symbol Type-C:USB_C_GCT_USB4085
- removed Y1: Crystal, cftkb:Crystal_HC49-4H_Vertical, symbol Device:Crystal
- added U1: Pro_Micro, keebio:ArduinoProMicro-TopSide, symbol Keyboard_Parts:Pro_Micro
- RESET1: symbol romeo-pcb-rescue:SW_PUSH-keyboard_parts -> juliet-pcb-rescue:SW_PUSH-keyboard_parts
- SW0, SW1, SW10, SW11, SW12, SW13, SW14, SW15, SW16, SW17, SW18, SW19, SW2, SW20, SW21, SW22, SW23, SW24, SW25, SW26, SW27, SW28, SW29, SW3, SW30, SW31, SW32, SW33, SW34, SW35, SW36, SW37, SW38, SW39, SW4, SW40, SW41, SW42, SW43, SW44, SW45, SW46, SW47, SW5, SW6, SW7, SW8, SW9: symbol keyboard_parts:KEYSW -> juliet-pcb-rescue:KEYSW-keyboard_parts
Connections:
- net labels added: RAW
- net labels removed: +5V, D+, D-, VCC, boot, sck, xtal1, xtal2
- wire segments 200 -> 151
- no-connect marks 3 -> 0
