File: juliet-pcb.kicad_pcb (KiCad board)
At the start: 2 copper layers, 247.6 x 99.2 mm, 104 parts, among them SW0 KEYSW, SW1 KEYSW, SW10 KEYSW, SW11 KEYSW, SW12 KEYSW, SW13 KEYSW, SW14 KEYSW, SW15 KEYSW, SW16 KEYSW, SW17 KEYSW, SW18 KEYSW, SW19 KEYSW, SW2 KEYSW, SW20 KEYSW, SW21 KEYSW, SW22 KEYSW, SW23 KEYSW, SW24 KEYSW, SW25 KEYSW, SW26 KEYSW, SW27 KEYSW, SW28 KEYSW, SW29 KEYSW, SW3 KEYSW, SW30 KEYSW, SW31 KEYSW, SW32 KEYSW, SW33 KEYSW, SW34 KEYSW, SW35 KEYSW, SW36 KEYSW, SW37 KEYSW, SW38 KEYSW, SW39 KEYSW, SW4 KEYSW, SW40 KEYSW, SW41 KEYSW, SW42 KEYSW, SW43 KEYSW, SW44 KEYSW, SW45 KEYSW, SW46 KEYSW, SW47 KEYSW, SW5 KEYSW, SW6 KEYSW, SW7 KEYSW, SW8 KEYSW, SW9 KEYSW, U1 Pro_Micro

Commit message: rev1
Parts:
- added G***: LOGO, Custom Footies:triangles_400, F.Cu at (240.4, 49.8)
- added G***: LOGO, Custom Footies:triangles_400, F.Cu at (52.7, 47.1)
- added G***: LOGO, Custom Footies:triangles_400, F.Cu at (242.9, 47.1)
- added G***: LOGO, Custom Footies:triangles_400, F.Cu at (55.3, 49.8)
- added G***: LOGO, juliet:juliet_logo_150_dpi, B.Cu at (189.6, 73.1)
Other:
- board text added: "GPLv3"
