File: juliet-pcb.kicad_pcb (KiCad board)
At the start: 2 copper layers, 247.6 x 99.2 mm, 109 parts, among them SW0 KEYSW, SW1 KEYSW, SW10 KEYSW, SW11 KEYSW, SW12 KEYSW, SW13 KEYSW, SW14 KEYSW, SW15 KEYSW, SW16 KEYSW, SW17 KEYSW, SW18 KEYSW, SW19 KEYSW, SW2 KEYSW, SW20 KEYSW, SW21 KEYSW, SW22 KEYSW, SW23 KEYSW, SW24 KEYSW, SW25 KEYSW, SW26 KEYSW, SW27 KEYSW, SW28 KEYSW, SW29 KEYSW, SW3 KEYSW, SW30 KEYSW, SW31 KEYSW, SW32 KEYSW, SW33 KEYSW, SW34 KEYSW, SW35 KEYSW, SW36 KEYSW, SW37 KEYSW, SW38 KEYSW, SW39 KEYSW, SW4 KEYSW, SW40 KEYSW, SW41 KEYSW, SW42 KEYSW, SW43 KEYSW, SW44 KEYSW, SW45 KEYSW, SW46 KEYSW, SW47 KEYSW, SW5 KEYSW, SW6 KEYSW, SW7 KEYSW, SW8 KEYSW, SW9 KEYSW, U1 Pro_Micro

Commit message: lol fixed
Connections:
- U1 pad 19: Net-(U1-Pad19) -> row3
- U1 pad 20: Net-(U1-Pad20) -> row0
- U1 pad 23: Net-(U1-Pad23) -> GND
- U1 pad 3: row0 -> GND
- U1 pad 4: row3 -> GND
Routing:
- net row0: track 238.8 -> 256.6 mm
- net row3: track 202.2 -> 217.8 mm
- net row2: track 211.5 -> 210.0 mm
- net row1: track 225.7 -> 224.8 mm, vias 0 -> 1

Commit message: Fixed the issues.
Routing:
- net row0: track 256.6 -> 239.3 mm
- net row2: track 210.0 -> 205.4 mm
- net row1: track 224.8 -> 222.2 mm
- net row3: track 217.8 -> 217.0 mm, vias 1 -> 0
