File: juliet-pcb.kicad_pcb (KiCad board)
At the start: 2 copper layers, 247.6 x 99.2 mm, 109 parts, among them SW0 KEYSW, SW1 KEYSW, SW10 KEYSW, SW11 KEYSW, SW12 KEYSW, SW13 KEYSW, SW14 KEYSW, SW15 KEYSW, SW16 KEYSW, SW17 KEYSW, SW18 KEYSW, SW19 KEYSW, SW2 KEYSW, SW20 KEYSW, SW21 KEYSW, SW22 KEYSW, SW23 KEYSW, SW24 KEYSW, SW25 KEYSW, SW26 KEYSW, SW27 KEYSW, SW28 KEYSW, SW29 KEYSW, SW3 KEYSW, SW30 KEYSW, SW31 KEYSW, SW32 KEYSW, SW33 KEYSW, SW34 KEYSW, SW35 KEYSW, SW36 KEYSW, SW37 KEYSW, SW38 KEYSW, SW39 KEYSW, SW4 KEYSW, SW40 KEYSW, SW41 KEYSW, SW42 KEYSW, SW43 KEYSW, SW44 KEYSW, SW45 KEYSW, SW46 KEYSW, SW47 KEYSW, SW5 KEYSW, SW6 KEYSW, SW7 KEYSW, SW8 KEYSW, SW9 KEYSW, U1 Pro_Micro

Commit message: Updated pro micro location
Parts:
- moved U1 34.2 mm to (200.7, 52.1)
Connections:
- net Net-(U1-Pad17) renamed NO-OP3
- net Net-(U1-Pad18) renamed NO-OP2
- net Net-(U1-Pad21) renamed NO-OP1
Routing:
- net reset: track 65.0 -> 99.6 mm
- net col0: track 202.4 -> 236.8 mm
- net col1: track 168.3 -> 202.7 mm
- net col4: track 120.7 -> 155.1 mm
- net col6: track 92.0 -> 126.4 mm
- net col5: track 84.2 -> 118.5 mm
- net col3: track 117.2 -> 151.6 mm
- net col2: track 155.1 -> 189.5 mm
- net col9: track 127.2 -> 95.1 mm
- net col10: track 136.2 -> 105.3 mm
- net col11: track 157.7 -> 127.7 mm
- net col7: track 77.4 -> 106.6 mm
- net row3: track 217.0 -> 243.8 mm
- net col8: track 90.4 -> 86.6 mm
- net row0: track 239.3 -> 238.2 mm, vias 0 -> 1
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
Commit message: Fixed a lot of issues.
Parts:
- added G***: LOGO, Custom Footies:triangles_400, F.Cu at (111.8, 49.8)
- added G***: LOGO, Custom Footies:triangles_400, F.Cu at (109.1, 47.1)
- added G***: LOGO, Custom Footies:triangles_400, F.Cu at (96.5, 49.8)
- added G***: LOGO, Custom Footies:triangles_400, F.Cu at (93.8, 47.1)
- moved RESET1 41.1 mm to (141.1, 49.2)
Connections:
- net NO-OP1 renamed Net-(U1-Pad21)
- net NO-OP2 renamed Net-(U1-Pad18)
- net NO-OP3 renamed Net-(U1-Pad17)
- U1 pad 19: row3 -> row0
- U1 pad 20: row0 -> row3
Routing:
- net reset: track 99.6 -> 58.5 mm
- net row3: track 243.8 -> 222.3 mm
- net row0: track 238.2 -> 239.9 mm, vias 1 -> 0
